File: stormduino Rev2.kicad_pcb (KiCad board)
At the start: 2 copper layers, 68.6 x 53.3 mm, 50 parts, among them J1 Jack-DC, J2 USB_C_Receptacle_USB2.0, J3 Conn_02x03_Odd_Even, J4 Conn_01x06_MountingPin, J5 Conn_01x08_MountingPin, J6 Conn_01x10_MountingPin, J7 Conn_01x08_MountingPin, Q1 BS250, SW1 SW_Push, U1 LM358, U2 AMS1117-5.0, U3 AMS1117-3.3, U4 CH340C, U5 ATmega328P-PU, Y1 16 Mhz

Commit message: Add files via upload
Parts:
- removed C5: 47uF, Capacitor_THT:CP_Radial_D5.0mm_P2.50mm
- removed the G*** at (128.6, 70.7)
- removed the REF** at (122.3, 77.3)
- added C2: 10uF, Capacitor_SMD:CP_Elec_6.3x5.4, F.Cu at (134.1, 88.0)
- added G***: LOGO, logo:modern-dodos-3, B.Cu at (139.8, 71.7)
- added J8: Conn_01x04_MountingPin, Connector_PinHeader_1.27mm:PinHeader_1x04_P1.27mm_Vertical, F.Cu at (133.8, 60.7)
- added J9: Conn_01x06_MountingPin, Connector_PinHeader_1.27mm:PinHeader_1x06_P1.27mm_Vertical, F.Cu at (122.1, 65.0)
- C1: footprint Capacitor_THT:CP_Radial_D5.0mm_P2.50mm -> Capacitor_SMD:CP_Elec_6.3x5.4
- moved G*** 14.1 mm to (138.3, 53.8)
- moved G*** 14.0 mm to (138.0, 67.4)
- moved C13 5.67 mm to (137.7, 81.8)
- moved C8 5.10 mm to (133.2, 65.8)
- moved R2 4.41 mm to (123.4, 78.5)
- moved C4 4.41 mm to (130.5, 81.9)
- moved C9 4.41 mm to (124.5, 70.2)
- moved U1 4.41 mm to (130.8, 77.9)
- moved C2 4.41 mm to (123.4, 76.1)
- moved C6 4.41 mm to (122.4, 70.2)
- moved C7 4.41 mm to (123.4, 74.0)
- moved R1 4.41 mm to (123.4, 80.6)
- moved C10 4.07 mm to (137.4, 73.4), turned to 0 degrees
- moved C1 1.30 mm to (125.9, 88.0), turned to 90 degrees
- moved J1 0.43 mm to (119.5, 91.4)
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Connections:
- U4 pad 10: Net-(U4-Pad10) -> /DSR
- U4 pad 11: Net-(U4-Pad11) -> /RI
- U4 pad 12: Net-(U4-Pad12) -> /DCD
- U4 pad 14: Net-(U4-Pad14) -> /RTS
- U4 pad 15: Net-(U4-Pad15) -> /R232
- U4 pad 9: Net-(U4-Pad9) -> /CTS
Routing:
- net /RTS: track 0.00 -> 9.83 mm, vias 0 -> 1
- net /R232: track 0.00 -> 8.77 mm, vias 0 -> 1
- net +5V: track 203.8 -> 212.2 mm, vias 4 -> 7
- net /AREF: track 87.9 -> 95.1 mm
- net GND: track 13.4 -> 7.95 mm
- net /D0: track 85.6 -> 90.8 mm
- net Net-(C8-Pad2): track 2.39 -> 6.86 mm
- net +3V3: track 85.5 -> 89.9 mm
- net /DCD: track 0.00 -> 3.24 mm
- net /DSR: track 0.00 -> 3.23 mm
- net /CTS: track 0.00 -> 3.23 mm
- net /RI: track 0.00 -> 3.23 mm
- net /D1: track 94.6 -> 97.2 mm
- net /D13: track 125.0 -> 127.7 mm
- net Net-(R5-Pad1): track 17.2 -> 14.6 mm
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Other:
- board text added: "CTS DSR RI DCD RTS R232"
- board text added: "REV 2.2"
- board text added: "VCC"
- board text removed: "MADE IN MAURITIUS"
- board text removed: "REV 2.1"
